File: output/pcbs/theboard.kicad_pcb (KiCad board)
At the start: 2 copper layers, 297.1 x 120.3 mm, 79 parts

Commit message: V1 - off to the printers
Parts:
- added _1: , MountingHole_2.2mm_M2_Pad_Via, F.Cu at (15.2, -50.6)
- added _10: , MountingHole_2.2mm_M2_Pad_Via, F.Cu at (153.8, 24.2)
- added _2: , MountingHole_2.2mm_M2_Pad_Via, F.Cu at (253.0, -50.6)
- added _3: , MountingHole_2.2mm_M2_Pad_Via, F.Cu at (5.40, -4.00)
- added _4: , MountingHole_2.2mm_M2_Pad_Via, F.Cu at (262.9, -4.00)
- added _5: , MountingHole_2.2mm_M2_Pad_Via, F.Cu at (76.4, 11.1)
- added _6: , MountingHole_2.2mm_M2_Pad_Via, F.Cu at (191.9, 11.1)
- added _7: , MountingHole_2.2mm_M2_Pad_Via, F.Cu at (119.5, -41.2)
- added _8: , MountingHole_2.2mm_M2_Pad_Via, F.Cu at (148.8, -41.2)
- added _9: , MountingHole_2.2mm_M2_Pad_Via, F.Cu at (114.5, 24.2)
- moved MCU1 3.31 mm to (132.9, -19.8), turned to 271.25 degrees
- moved OLED1 3.29 mm to (128.1, -0.81)
- moved S38 2.30 mm to (159.6, 38.0), turned to 41.25 degrees
- moved S19 2.27 mm to (108.6, 38.0), turned to -41.25 degrees
- moved D38 2.23 mm to (162.9, 41.8), turned to 41.25 degrees
- moved D19 2.20 mm to (105.4, 41.8), turned to -41.25 degrees
- moved S36 2.04 mm to (158.4, -29.7), turned to 21.25 degrees
- moved S17 1.99 mm to (109.9, -29.7), turned to -21.25 degrees
- moved D36 1.98 mm to (160.2, -25.0), turned to 21.25 degrees
- moved D17 1.94 mm to (108.1, -25.0), turned to -21.25 degrees
- moved S35 1.84 mm to (165.2, -12.0), turned to 21.25 degrees
- moved S16 1.81 mm to (103.0, -12.0), turned to -21.25 degrees
- moved S33 1.80 mm to (177.3, -39.2), turned to 18.25 degrees
- moved D35 1.79 mm to (167.1, -7.32), turned to 21.25 degrees
- moved D16 1.77 mm to (101.2, -7.32), turned to -21.25 degrees
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Other:
- board size 297.1 x 120.3 mm -> 298.5 x 123.3 mm
