File: thesplit/thesplit.kicad_pcb (KiCad board)
At the start: 2 copper layers, 297.1 x 120.3 mm, 79 parts

Commit message: local ergogen
Parts:
- moved S10 302.4 mm to (251.8, 191.5)
- moved S13 302.4 mm to (268.1, 202.9)
- moved S17 302.4 mm to (292.9, 193.9)
- moved S2 302.4 mm to (188.5, 187.8)
- moved D1 302.4 mm to (185.4, 211.6)
- moved D12 302.4 mm to (261.0, 225.8)
- moved D13 302.4 mm to (266.7, 207.7)
- moved D18 302.4 mm to (270.8, 253.9)
- moved D24 302.4 mm to (424.2, 186.9)
- moved D29 302.4 mm to (385.2, 196.3)
- moved D32 302.4 mm to (368.9, 207.7)
- moved D6 302.4 mm to (225.3, 214.7)
- moved D9 302.4 mm to (244.7, 214.4)
- moved S19 302.4 mm to (291.9, 261.3)
- moved S20 302.4 mm to (449.5, 206.6)
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Connections:
- D1 pad 1: (no net) -> P15
- D10 pad 1: (no net) -> P15
- D11 pad 1: (no net) -> P21
- D12 pad 1: (no net) -> P16
- D13 pad 1: (no net) -> P15
- D14 pad 1: (no net) -> P21
- D15 pad 1: (no net) -> P16
- D16 pad 1: (no net) -> P15
- D17 pad 1: (no net) -> P21
- D18 pad 1: (no net) -> P10
- D19 pad 1: (no net) -> P10
- D2 pad 1: (no net) -> P21
- D20 pad 1: (no net) -> P6
- D21 pad 1: (no net) -> P1
- D22 pad 1: (no net) -> P8
- D23 pad 1: (no net) -> P6
- D24 pad 1: (no net) -> P1
- D25 pad 1: (no net) -> P8
- D26 pad 1: (no net) -> P6
- D27 pad 1: (no net) -> P1
- D28 pad 1: (no net) -> P8
- D29 pad 1: (no net) -> P6
- D3 pad 1: (no net) -> P16
- D30 pad 1: (no net) -> P1
- D31 pad 1: (no net) -> P8
- D32 pad 1: (no net) -> P6
- D33 pad 1: (no net) -> P1
- D34 pad 1: (no net) -> P8
- D35 pad 1: (no net) -> P6
- D36 pad 1: (no net) -> P1
- D37 pad 1: (no net) -> P9
- D38 pad 1: (no net) -> P9
- D4 pad 1: (no net) -> P15
- D5 pad 1: (no net) -> P21
- D6 pad 1: (no net) -> P16
- D7 pad 1: (no net) -> P15
- D8 pad 1: (no net) -> P21
- D9 pad 1: (no net) -> P16
- S1 pad 1: (no net) -> P20
- S10 pad 1: (no net) -> P14
- S11 pad 1: (no net) -> P14
- S12 pad 1: (no net) -> P4
- S13 pad 1: (no net) -> P4
- S14 pad 1: (no net) -> P4
- S15 pad 1: (no net) -> P3
- S16 pad 1: (no net) -> P3
- S17 pad 1: (no net) -> P3
- S18 pad 1: (no net) -> P4
- S19 pad 1: (no net) -> P3
- S2 pad 1: (no net) -> P20
- S20 pad 1: (no net) -> P20
- S21 pad 1: (no net) -> P20
- S22 pad 1: (no net) -> P19
- S23 pad 1: (no net) -> P19
- S24 pad 1: (no net) -> P19
- S25 pad 1: (no net) -> p18
- S26 pad 1: (no net) -> p18
- S27 pad 1: (no net) -> p18
- S28 pad 1: (no net) -> P14
- S29 pad 1: (no net) -> P14
- S3 pad 1: (no net) -> P19
- S30 pad 1: (no net) -> P14
- S31 pad 1: (no net) -> P4
- S32 pad 1: (no net) -> P4
- S33 pad 1: (no net) -> P4
- S34 pad 1: (no net) -> P3
- S35 pad 1: (no net) -> P3
- S36 pad 1: (no net) -> P3
- S37 pad 1: (no net) -> P4
- S38 pad 1: (no net) -> P3
- S4 pad 1: (no net) -> P19
- S5 pad 1: (no net) -> P19
- S6 pad 1: (no net) -> p18
- S7 pad 1: (no net) -> p18
- S8 pad 1: (no net) -> p18
- S9 pad 1: (no net) -> P14
Routing:
- net p18: track 0.00 -> 336.1 mm
- net P20: track 0.00 -> 335.1 mm
- net P19: track 0.00 -> 318.1 mm
- net P14: track 0.00 -> 310.6 mm
- net P4: track 0.00 -> 269.2 mm
- net P3: track 0.00 -> 234.9 mm
- net P15: track 0.00 -> 129.6 mm
- net P21: track 0.00 -> 129.3 mm
- net P1: track 0.00 -> 128.3 mm
- net P6: track 0.00 -> 124.6 mm
- net P16: track 0.00 -> 99.8 mm
- net P8: track 0.00 -> 93.2 mm
- net GND: track 0.00 -> 65.9 mm
- net RST: track 0.00 -> 34.2 mm
- net VCC: track 0.00 -> 26.7 mm
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
Commit message: V1 - off to the printers
Parts:
- removed OLED1: OLED, lib:OLED_headers
- added G***: LOGO, myboard:pcb-graphic-2, F.Cu at (342.0, 247.0)
- added _1: , MountingHole_2.2mm_M2_Pad_Via, F.Cu at (223.3, 174.3)
- added _10: , MountingHole_2.2mm_M2_Pad_Via, F.Cu at (361.9, 249.1)
- added _2: , MountingHole_2.2mm_M2_Pad_Via, F.Cu at (461.1, 174.3)
- added _3: , MountingHole_2.2mm_M2_Pad_Via, F.Cu at (213.5, 220.9)
- added _4: , MountingHole_2.2mm_M2_Pad_Via, F.Cu at (471.0, 220.9)
- added _5: , MountingHole_2.2mm_M2_Pad_Via, F.Cu at (284.5, 236.0)
- added _6: , MountingHole_2.2mm_M2_Pad_Via, F.Cu at (400.0, 236.0)
- added _7: , MountingHole_2.2mm_M2_Pad_Via, F.Cu at (327.6, 183.7)
- added _8: , MountingHole_2.2mm_M2_Pad_Via, F.Cu at (356.9, 183.7)
- added _9: , MountingHole_2.2mm_M2_Pad_Via, F.Cu at (322.6, 249.1)
- moved S8 25.5 mm to (261.3, 173.3), turned to -15.25 degrees
- moved S11 25.5 mm to (282.9, 174.1), turned to -18.25 degrees
- moved D8 25.4 mm to (260.0, 178.2), turned to -15.25 degrees
- moved D11 25.4 mm to (281.3, 178.8), turned to -18.25 degrees
- moved S5 25.3 mm to (237.7, 182.0), turned to -13.25 degrees
- moved S14 25.3 mm to (299.0, 185.7), turned to -18.25 degrees
- moved D5 25.2 mm to (236.6, 186.8), turned to -13.25 degrees
- moved S2 25.2 mm to (213.7, 187.3), turned to -8.5 degrees
- moved D14 25.2 mm to (297.5, 190.5), turned to -18.25 degrees
- moved S10 25.1 mm to (276.9, 192.1), turned to -18.25 degrees
- moved S7 25.1 mm to (256.3, 191.7), turned to -15.25 degrees
- moved D2 25.1 mm to (213.0, 192.3), turned to -8.5 degrees
- moved S17 25.1 mm to (318.0, 195.2), turned to -21.25 degrees
- moved D10 25.1 mm to (275.4, 196.9), turned to -18.25 degrees
- moved D7 25.1 mm to (255.0, 196.5), turned to -15.25 degrees
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Connections:
- S25 pad 1: p18 -> P18
- S26 pad 1: p18 -> P18
- S27 pad 1: p18 -> P18
- S6 pad 1: p18 -> P18
- S7 pad 1: p18 -> P18
- S8 pad 1: p18 -> P18
Routing:
- net P18: track 0.00 -> 468.0 mm, vias 0 -> 1
- net p18: track 336.1 -> 0.00 mm
- net P20: track 335.1 -> 530.9 mm, vias 0 -> 1
- net P19: track 318.1 -> 499.9 mm, vias 0 -> 1
- net P14: track 310.6 -> 415.1 mm, vias 0 -> 1
- net P10: track 23.8 -> 101.1 mm
- net P16: track 99.8 -> 176.0 mm
- net P9: track 24.1 -> 100.2 mm
- net P15: track 129.6 -> 192.6 mm, vias 0 -> 2
- net P8: track 93.2 -> 152.7 mm
- net P21: track 129.3 -> 186.5 mm, vias 0 -> 2
- net P4: track 269.2 -> 320.1 mm, vias 0 -> 1
- net P6: track 124.6 -> 170.8 mm
- net P1: track 128.3 -> 172.2 mm
- net P3: track 234.9 -> 262.7 mm, vias 0 -> 1
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Other:
- board size 297.1 x 120.3 mm -> 298.3 x 123.3 mm
- board text added: "Jingis 38 v1.0.0"
